Commit message: Avoid gliding: change caster joints to continuous

File: kobuki_description/urdf/kobuki.urdf.xacro (robot description, xacro)
@@ -61,4 +61,5 @@
       <origin xyz="0.00 ${0.23/2} 0.0250" rpy="${-M_PI/2} 0 0"/>
       <axis xyz="0 0 1"/>
+      <!--<dynamics damping="0.0" friction="0.1"/>-->
     </joint>
     <link name="wheel_left_link">
@@ -78,7 +79,7 @@
         <mass value="0.01" />
         <origin xyz="0 0 0" />
-        <inertia ixx="0.001" ixy="0.0" ixz="0.0"
-                 iyy="0.001" iyz="0.0"
-                 izz="0.001" />
+        <inertia ixx="0.00001" ixy="0.0" ixz="0.0"
+                 iyy="0.00001" iyz="0.0"
+                 izz="0.00001" />
       </inertial>
     </link>
@@ -88,4 +89,5 @@
       <origin xyz="0.00 -${0.23/2} 0.0250" rpy="${-M_PI/2} 0 0"/>
       <axis xyz="0 0 1"/>
+      <!--<dynamics damping="0.0" friction="0.1"/>-->
     </joint>
     <link name="wheel_right_link">
@@ -105,47 +107,49 @@
         <mass value="0.01" />
         <origin xyz="0 0 0" />
-        <inertia ixx="0.001" ixy="0.0" ixz="0.0"
-                 iyy="0.001" iyz="0.0"
-                 izz="0.001" />
-      </inertial>
-    </link>
-    <joint name="caster_front_joint" type="fixed">
+        <inertia ixx="0.00001" ixy="0.0" ixz="0.0"
+                 iyy="0.00001" iyz="0.0"
+                 izz="0.00001" />
+      </inertial>
+    </link>
+    <joint name="caster_front_joint" type="continuous">
       <parent link="base_link"/>
       <child link="caster_front_link"/>
       <origin xyz="0.115 0.0 0.007" rpy="${-M_PI/2} 0 0"/>
+      <axis xyz="0 0 1"/>
     </joint>
     <link name="caster_front_link">
       <collision>
         <geometry>
-          <cylinder length="0.0176" radius="0.017"/>
-        </geometry>
-        <origin rpy="0 0 0" xyz="0 0 0"/>
-      </collision>
-      <inertial>
-        <mass value="0.01" />
-        <origin xyz="0 0 0" />
-        <inertia ixx="0.001" ixy="0.0" ixz="0.0"
-                 iyy="0.001" iyz="0.0"
-                 izz="0.001" />
-      </inertial>
-    </link>
-    <joint name="caster_back_joint" type="fixed">
+          <sphere radius="0.017"/>
+        </geometry>
+        <origin rpy="0 0 0" xyz="0 0 0"/>
+      </collision>
+      <inertial>
+        <mass value="0.01" />
+        <origin xyz="0 0 0" />
+        <inertia ixx="0.000001" ixy="0.0" ixz="0.0"
+                 iyy="0.000001" iyz="0.0"
+                 izz="0.000001" />
+      </inertial>
+    </link>
+    <joint name="caster_back_joint" type="continuous">
       <parent link="base_link"/>
       <child link="caster_back_link"/>
       <origin xyz="-0.135 0.0 0.009" rpy="${-M_PI/2} 0 0"/>
+      <axis xyz="0 0 1"/>
     </joint>
     <link name="caster_back_link">
       <collision>
         <geometry>
-          <cylinder length="0.0176" radius="0.017"/>
-        </geometry>
-        <origin rpy="0 0 0" xyz="0 0 0"/>
-      </collision>
-      <inertial>
-        <mass value="0.01" />
-        <origin xyz="0 0 0" />
-        <inertia ixx="0.001" ixy="0.0" ixz="0.0"
-                 iyy="0.001" iyz="0.0"
-                 izz="0.001" />
+          <sphere radius="0.017"/>
+        </geometry>
+        <origin rpy="0 0 0" xyz="0 0 0"/>
+      </collision>
+      <inertial>
+        <mass value="0.01" />
+        <origin xyz="0 0 0" />
+        <inertia ixx="0.000001" ixy="0.0" ixz="0.0"
+                 iyy="0.000001" iyz="0.0"
+                 izz="0.000001" />
       </inertial>
     </link>

File: kobuki_description/urdf/kobuki_gazebo.urdf.xacro (robot description, xacro)
@@ -2,7 +2,15 @@
 <robot name="kobuki_sim" xmlns:xacro="http://ros.org/wiki/xacro">
   <xacro:macro name="kobuki_sim">
+<!--    <gazebo reference="wheel_left_joint">
+      <implicitSpringDamper>1</implicitSpringDamper>
+      <springStiffness>1</springStiffness>
+    </gazebo>
+    <gazebo reference="wheel_right_joint">
+      <implicitSpringDamper>1</implicitSpringDamper>
+      <springStiffness>1</springStiffness>
+    </gazebo>-->
     <gazebo reference="wheel_left_link">
-      <mu1>1.0</mu1>
-      <mu2>1.0</mu2>
+      <mu1>200.0</mu1>
+      <mu2>100.0</mu2>
       <kp>1000000.0</kp>
       <kd>100.0</kd>
@@ -11,6 +19,6 @@
     </gazebo>
     <gazebo reference="wheel_right_link">
-      <mu1>1.0</mu1>
-      <mu2>1.0</mu2>
+      <mu1>200.0</mu1>
+      <mu2>100.0</mu2>
       <kp>1000000.0</kp>
       <kd>100.0</kd>
@@ -23,5 +31,5 @@
       <kp>1000000.0</kp>
       <kd>100.0</kd>
-      <minDepth>0.001</minDepth>
+      <minDepth>0.0</minDepth>
       <maxVel>1.0</maxVel>
     </gazebo>
@@ -31,5 +39,5 @@
       <kp>1000000.0</kp>
       <kd>100.0</kd>
-      <minDepth>0.001</minDepth>
+      <minDepth>0.0</minDepth>
       <maxVel>1.0</maxVel>
     </gazebo>

Commit message: Calculate more realistic inertia tensors using a cylindric model Use a sphere as collision model for the caster wheels (one contact point)

File: kobuki_description/urdf/kobuki.urdf.xacro (robot description, xacro)
@@ -9,4 +9,15 @@
   <xacro:include filename="$(find kobuki_description)/urdf/common_properties.urdf.xacro"/>
   <xacro:include filename="$(find kobuki_description)/urdf/kobuki_gazebo.urdf.xacro"/>
+  <!-- Inertia tensor of a cylinder with homogeneous mass distribution. From
+       https://en.wikipedia.org/wiki/List_of_moments_of_inertia#List_of_3D_inertia_tensors-->
+  <xacro:macro name="cylinder_inertia" params="radius height mass x=0 y=0 z=0">
+    <inertial>
+      <mass value="${mass}"/>
+      <origin xyz="${x} ${y} ${z}"/>
+      <inertia ixx="${1/12 * mass * (3 * radius**2 + height**2)}" ixy="0" ixz="0"
+               iyy="${1/12 * mass * (3 * radius**2 + height**2)}" iyz="0"
+               izz="${1/2 * mass * radius**2}"/>
+    </inertial>
+  </xacro:macro>
   <!-- Kobuki -->
   <xacro:macro name="kobuki">
@@ -29,5 +40,4 @@
       <visual>
         <geometry>
-          <!-- new mesh -->
           <mesh filename="package://kobuki_description/meshes/main_body.dae" />
         </geometry>
@@ -40,19 +50,11 @@
         <origin xyz="0.0 0 0.05949" rpy="0 0 0"/>
       </collision>
-      <inertial>
-        <!-- COM experimentally determined -->
-        <origin xyz="0.01 0 0"/>
-        <mass value="2.4"/> <!-- 2.4/2.6 kg for small/big battery pack -->
         <!-- Kobuki's inertia tensor is approximated by a cylinder with homogeneous mass distribution
-             More details: http://en.wikipedia.org/wiki/List_of_moment_of_inertia_tensors
-             m = 2.4 kg; h = 0.09 m; r = 0.175 m
-             ixx = 1/12 * m * (3 * r^2 + h^2)
-             iyy = 1/12 * m * (3 * r^2 + h^2)
-             izz = 1/2 * m * r^2
+             m = 2.4 kg (2.6 kg for big battery pack); h = 0.09 m; r = 0.175 m; COM experimentally determined
+             ixx = 1/12 * m * (3 * r^2 + h^2) = 0.019995
+             iyy = 1/12 * m * (3 * r^2 + h^2) = 0.019995
+             izz = 1/2 * m * r^2 = 0.03675
           -->
-        <inertia ixx="0.019995" ixy="0.0" ixz="0.0"
-                 iyy="0.019995" iyz="0.0"
-                 izz="0.03675" />
-      </inertial>
+      <xacro:cylinder_inertia radius="0.175" height="0.09" mass="2.4" x="0.01" z="0.03"/>
     </link>
     <joint name="wheel_left_joint" type="continuous">
@@ -75,11 +77,5 @@
         <origin rpy="0 0 0" xyz="0 0 0"/>
       </collision>
-      <inertial>
-        <mass value="0.01" />
-        <origin xyz="0 0 0" />
-        <inertia ixx="0.001" ixy="0.0" ixz="0.0"
-                 iyy="0.001" iyz="0.0"
-                 izz="0.001" />
-      </inertial>
+      <xacro:cylinder_inertia radius="0.035" height="0.0206" mass="0.15"/>
     </link>
     <joint name="wheel_right_joint" type="continuous">
@@ -102,11 +98,5 @@
         <origin rpy="0 0 0" xyz="0 0 0"/>
       </collision>
-      <inertial>
-        <mass value="0.01" />
-        <origin xyz="0 0 0" />
-        <inertia ixx="0.001" ixy="0.0" ixz="0.0"
-                 iyy="0.001" iyz="0.0"
-                 izz="0.001" />
-      </inertial>
+      <xacro:cylinder_inertia radius="0.035" height="0.0206" mass="0.15"/>
     </link>
     <joint name="caster_front_joint" type="fixed">
@@ -118,15 +108,9 @@
       <collision>
         <geometry>
-          <cylinder length="0.0176" radius="0.017"/>
+          <sphere radius="0.017"/>
         </geometry>
         <origin rpy="0 0 0" xyz="0 0 0"/>
       </collision>
-      <inertial>
-        <mass value="0.01" />
-        <origin xyz="0 0 0" />
-        <inertia ixx="0.001" ixy="0.0" ixz="0.0"
-                 iyy="0.001" iyz="0.0"
-                 izz="0.001" />
-      </inertial>
+      <xacro:cylinder_inertia radius="0.017" height="0.0176" mass="0.005"/>
     </link>
     <joint name="caster_back_joint" type="fixed">
@@ -138,15 +122,9 @@
       <collision>
         <geometry>
-          <cylinder length="0.0176" radius="0.017"/>
+          <sphere radius="0.017"/>
         </geometry>
         <origin rpy="0 0 0" xyz="0 0 0"/>
       </collision>
-      <inertial>
-        <mass value="0.01" />
-        <origin xyz="0 0 0" />
-        <inertia ixx="0.001" ixy="0.0" ixz="0.0"
-                 iyy="0.001" iyz="0.0"
-                 izz="0.001" />
-      </inertial>
+      <xacro:cylinder_inertia radius="0.017" height="0.0176" mass="0.005"/>
     </link>
     <!-- Kobuki's sensors -->

Commit message: Partially revert: spherical wheels don't avoid drift, and motor wheels need huge inertias

File: kobuki_description/urdf/kobuki.urdf.xacro (robot description, xacro)
@@ -77,5 +77,13 @@
         <origin rpy="0 0 0" xyz="0 0 0"/>
       </collision>
-      <xacro:cylinder_inertia radius="0.035" height="0.0206" mass="0.15"/>
+      <inertial>
+        <mass value="0.15" />
+        <origin xyz="0 0 0" />
+        <!-- We cannot use cylinder_inertia macro cause we need huge inertia to make the model
+             work, hence the unrealistic mass of 5 (mass = 5.0, radius = 0.035, height = 0.0206) -->
+        <inertia ixx="${1/12 * 5.0 * (3 * 0.035**2 + 0.0206**2)}" ixy="0" ixz="0"
+                 iyy="${1/12 * 5.0 * (3 * 0.035**2 + 0.0206**2)}" iyz="0"
+                 izz="${1/2 * 5.0 * 0.035**2}"/>
+      </inertial>
     </link>
     <joint name="wheel_right_joint" type="continuous">
@@ -98,5 +106,12 @@
         <origin rpy="0 0 0" xyz="0 0 0"/>
       </collision>
-      <xacro:cylinder_inertia radius="0.035" height="0.0206" mass="0.15"/>
+      <inertial>
+        <mass value="0.15" />
+        <origin xyz="0 0 0" />
+        <!-- same as left wheel -->
+        <inertia ixx="${1/12 * 5.0 * (3 * 0.035**2 + 0.0206**2)}" ixy="0" ixz="0"
+                 iyy="${1/12 * 5.0 * (3 * 0.035**2 + 0.0206**2)}" iyz="0"
+                 izz="${1/2 * 5.0 * 0.035**2}"/>
+      </inertial>
     </link>
     <joint name="caster_front_joint" type="fixed">
@@ -108,5 +123,5 @@
       <collision>
         <geometry>
-          <sphere radius="0.017"/>
+          <cylinder length="0.0176" radius="0.017"/>
         </geometry>
         <origin rpy="0 0 0" xyz="0 0 0"/>
@@ -122,5 +137,5 @@
       <collision>
         <geometry>
-          <sphere radius="0.017"/>
+          <cylinder length="0.0176" radius="0.017"/>
         </geometry>
         <origin rpy="0 0 0" xyz="0 0 0"/>

Commit message: Add euler angles to cylinder_inertia macro

File: kobuki_description/urdf/kobuki.urdf.xacro (robot description, xacro)
@@ -11,8 +11,8 @@
   <!-- Inertia tensor of a cylinder with homogeneous mass distribution. From
        https://en.wikipedia.org/wiki/List_of_moments_of_inertia#List_of_3D_inertia_tensors-->
-  <xacro:macro name="cylinder_inertia" params="radius height mass x=0 y=0 z=0">
+  <xacro:macro name="cylinder_inertia" params="radius height mass x=0 y=0 z=0 R=0 P=0 Y=0">
     <inertial>
       <mass value="${mass}"/>
-      <origin xyz="${x} ${y} ${z}"/>
+      <origin xyz="${x} ${y} ${z}" rpy="${R} ${P} ${Y}"/>
       <inertia ixx="${1/12 * mass * (3 * radius**2 + height**2)}" ixy="0" ixz="0"
                iyy="${1/12 * mass * (3 * radius**2 + height**2)}" iyz="0"
